File: pcb/headlamp.kicad_pcb (KiCad board)
At the start: 2 copper layers, 34 x 34 mm, 60 parts, among them IC1 ATTINY841-SSU, P1 POWER, P2 SERIAL, P3 ISP, Q1 VEMT3700-GS08, Q2 NX2301P, Q3 DMP2035U, Q4 DMP2035U, SW1 BT2, SW2 BT1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

Commit message: Final schematic values, pcb
Parts:
- R20, R21: value 10k -> 12k
- R22, R23: value 82k -> 270k
Changed lines of the file:
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@@
     (links 117)
     (no_connects 0)
-    (area 120.270599 89.777899 164.031601 130.871901)
+    (area 124.105199 92.444099 158.241201 126.580101)
     (thickness 1.6)
     (drawings 19)
@@
   )
   (layers
-    (0 F.Cu signal hide)
-    (31 B.Cu signal)
+    (0 F.Cu signal)
+    (31 B.Cu signal hide)
     (32 B.Adhes user)
     (33 F.Adhes user)
@@
       (effects (font (size 1 1) (thickness 0.15)))
     )
-    (fp_text value 82k (at 0 1.9 90) (layer F.Fab)
+    (fp_text value 270k (at 0 1.9 90) (layer F.Fab)
       (effects (font (size 1 1) (thickness 0.15)))
     )
@@
       (effects (font (size 1 1) (thickness 0.15)))
     )
-    (fp_text value 10k (at 0 1.9 90) (layer F.Fab)
+    (fp_text value 12k (at 0 1.9 90) (layer F.Fab)
       (effects (font (size 1 1) (thickness 0.15)))
     )
@@
       (effects (font (size 1 1) (thickness 0.15)))
     )
-    (fp_text value 10k (at 0 1.9 90) (layer F.Fab)
+    (fp_text value 12k (at 0 1.9 90) (layer F.Fab)
       (effects (font (size 1 1) (thickness 0.15)))
     )
@@
       (effects (font (size 1 1) (thickness 0.15)))
     )
-    (fp_text value 82k (at 0 1.9 180) (layer F.Fab)
+    (fp_text value 270k (at 0 1.9 180) (layer F.Fab)
       (effects (font (size 1 1) (thickness 0.15)))
     )
@@
     (connect_pads (clearance 0.4))
     (min_thickness 0.05)
-    (fill yes (arc_segments 16) (thermal_gap 0.508) (thermal_bridge_width 0.508))
+    (fill (arc_segments 16) (thermal_gap 0.508) (thermal_bridge_width 0.508))
     (polygon
       (pts

Commit message: Updated capacitors values
Parts:
- C10, C9: value 100n -> 10n
- C4, C7, C8: value 100n -> 1u
- R10, R11: value 120 -> 220
Changed lines of the file:
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@@
     (links 117)
     (no_connects 0)
-    (area 124.105199 92.444099 158.241201 126.580101)
+    (area 120.270599 89.777899 164.031601 130.871901)
     (thickness 1.6)
     (drawings 19)
@@
   (layers
     (0 F.Cu signal)
-    (31 B.Cu signal hide)
+    (31 B.Cu signal)
     (32 B.Adhes user)
     (33 F.Adhes user)
@@
       (effects (font (size 1 1) (thickness 0.15)))
     )
-    (fp_text value 100n (at 0 1.9 180) (layer F.Fab)
+    (fp_text value 1u (at 0 1.9 180) (layer F.Fab)
       (effects (font (size 1 1) (thickness 0.15)))
     )
@@
       (effects (font (size 1 1) (thickness 0.15)))
     )
-    (fp_text value 100n (at 0 1.9 180) (layer F.Fab)
+    (fp_text value 1u (at 0 1.9 180) (layer F.Fab)
       (effects (font (size 1 1) (thickness 0.15)))
     )
@@
       (effects (font (size 1 1) (thickness 0.15)))
     )
-    (fp_text value 100n (at 0 1.9 180) (layer F.Fab)
+    (fp_text value 1u (at 0 1.9 180) (layer F.Fab)
       (effects (font (size 1 1) (thickness 0.15)))
     )
@@
       (effects (font (size 1 1) (thickness 0.15)))
     )
-    (fp_text value 100n (at 0 1.9 220) (layer F.Fab)
+    (fp_text value 10n (at 0 1.9 220) (layer F.Fab)
       (effects (font (size 1 1) (thickness 0.15)))
     )
@@
       (effects (font (size 1 1) (thickness 0.15)))
     )
-    (fp_text value 120 (at 0 1.9 90) (layer F.Fab)
+    (fp_text value 220 (at 0 1.9 90) (layer F.Fab)
       (effects (font (size 1 1) (thickness 0.15)))
     )
@@
       (effects (font (size 1 1) (thickness 0.15)))
     )
-    (fp_text value 120 (at 0 1.9 180) (layer F.Fab)
+    (fp_text value 220 (at 0 1.9 180) (layer F.Fab)
       (effects (font (size 1 1) (thickness 0.15)))
     )
@@
       (effects (font (size 1 1) (thickness 0.15)))
     )
-    (fp_text value 100n (at 0 1.9 180) (layer F.Fab)
+    (fp_text value 10n (at 0 1.9 180) (layer F.Fab)
       (effects (font (size 1 1) (thickness 0.15)))
     )
@@
     (connect_pads (clearance 0.4))
     (min_thickness 0.05)
-    (fill (arc_segments 16) (thermal_gap 0.508) (thermal_bridge_width 0.508))
+    (fill yes (arc_segments 16) (thermal_gap 0.508) (thermal_bridge_width 0.508))
     (polygon
       (pts

Commit message: Replaced diode by resistor - was causing rising mcu VCC from spikes on power lines
Parts:
- removed D1: RB751VM, Diodes_SMD:SOD-323
- added R26: 33, Resistors_SMD:R_0603, F.Cu at (154.5, 118.6)
- D6, D7: value CREE_XP-G3 -> LED
- R1, R7: value 10k -> 8k2
Changed lines of the file:
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@@
-(kicad_pcb (version 4) (host pcbnew 4.0.5)
+(kicad_pcb (version 4) (host pcbnew 4.0.6)
   (general
     (links 117)
     (no_connects 0)
-    (area 120.270599 89.777899 164.031601 130.871901)
+    (area 124.105199 92.444099 158.241201 126.580101)
     (thickness 1.6)
     (drawings 19)
-    (tracks 682)
+    (tracks 683)
     (zones 0)
     (modules 60)
@@
   (layers
     (0 F.Cu signal)
-    (31 B.Cu signal)
+    (31 B.Cu signal hide)
     (32 B.Adhes user)
     (33 F.Adhes user)
@@
   )
   (setup
-    (last_trace_width 0.25)
+    (last_trace_width 0.6)
     (user_trace_width 0.4)
     (user_trace_width 0.5)
@@
   )
   (module Diodes_SMD:SOD-323 (layer F.Cu)
-    (at 154.38 118.55 45)
-    (descr SOD-323)
-    (tags SOD-323)
-    (attr smd)
-    (fp_text reference D1 (at 0 -1.85 45) (layer F.SilkS) hide
-      (effects (font (size 1 1) (thickness 0.15)))
-    )
-    (fp_text value RB751VM (at 0.1 1.9 45) (layer F.Fab)
-      (effects (font (size 1 1) (thickness 0.15)))
-    )
-    (fp_line (start 0.2 0) (end 0.45 0) (layer F.Fab) (width 0.15))
-    (fp_line (start 0.2 0.35) (end -0.3 0) (layer F.Fab) (width 0.15))
-    (fp_line (start 0.2 -0.35) (end 0.2 0.35) (layer F.Fab) (width 0.15))
-    (fp_line (start -0.3 0) (end 0.2 -0.35) (layer F.Fab) (width 0.15))
-    (fp_line (start -0.3 0) (end -0.5 0) (layer F.Fab) (width 0.15))
-    (fp_line (start -0.3 -0.35) (end -0.3 0.35) (layer F.Fab) (width 0.15))
-    (fp_line (start -0.85 0.65) (end -0.85 -0.65) (layer F.Fab) (width 0.15))
-    (fp_line (start 0.85 0.65) (end -0.85 0.65) (layer F.Fab) (width 0.15))
-    (fp_line (start 0.85 -0.65) (end 0.85 0.65) (layer F.Fab) (width 0.15))
-    (fp_line (start -0.85 -0.65) (end 0.85 -0.65) (layer F.Fab) (width 0.15))
-    (fp_line (start -1.5 -0.95) (end 1.5 -0.95) (layer F.CrtYd) (width 0.05))
-    (fp_line (start 1.5 -0.95) (end 1.5 0.95) (layer F.CrtYd) (width 0.05))
-    (fp_line (start -1.5 0.95) (end 1.5 0.95) (layer F.CrtYd) (width 0.05))
-    (fp_line (start -1.5 -0.95) (end -1.5 0.95) (layer F.CrtYd) (width 0.05))
-    (fp_line (start -1.3 0.8) (end 1.1 0.8) (layer F.SilkS) (width 0.15))
-    (fp_line (start -1.3 -0.8) (end 1.1 -0.8) (layer F.SilkS) (width 0.15))
-    (pad 1 smd rect (at -1.055 0 45) (size 0.59 0.45) (layers F.Cu F.Paste F.Mask)
-      (net 4 +3V3))
-    (pad 2 smd rect (at 1.055 0 45) (size 0.59 0.45) (layers F.Cu F.Paste F.Mask)
-      (net 1 VCC))
-    (model Diodes_SMD.3dshapes/SOD-323.wrl
-      (at (xyz 0 0 0))
-      (scale (xyz 1 1 1))
-      (rotate (xyz 0 0 180))
-    )
-  )
-  (module Diodes_SMD:SOD-323 (layer F.Cu)
     (at 155.702 112.014)
     (descr SOD-323)
@@
       (effects (font (size 1 1) (thickness 0.15)))
     )
-    (fp_text value 10k (at 0 1.9 270) (layer F.Fab)
+    (fp_text value 8k2 (at 0 1.9 270) (layer F.Fab)
       (effects (font (size 1 1) (thickness 0.15)))
     )
@@
       (effects (font (size 1 1) (thickness 0.15)))
     )
-    (fp_text value 10k (at 0 1.9) (layer F.Fab)
+    (fp_text value 8k2 (at 0 1.9) (layer F.Fab)
       (effects (font (size 1 1) (thickness 0.15)))
     )
@@
       (effects (font (size 1 1) (thickness 0.15)))
     )
-    (fp_text value CREE_XP-G3 (at 0 -1.8) (layer F.Fab)
+    (fp_text value LED (at 0 -1.8) (layer F.Fab)
       (effects (font (size 1 1) (thickness 0.15)))
     )
@@
       (effects (font (size 1 1) (thickness 0.15)))
     )
-    (fp_text value CREE_XP-G3 (at 0 -1.8 45) (layer F.Fab)
+    (fp_text value LED (at 0 -1.8 45) (layer F.Fab)
       (effects (font (size 1 1) (thickness 0.15)))
     )
@@
       (xy -0.026262 5.547126) (xy 0 5.547126) (xy 0.209014 5.547002)) (layer B.SilkS) (width 0.01))
   )
+  (module Resistors_SMD:R_0603 (layer F.Cu)
+    (at 154.4828 118.55196 45)
+    (descr "Resistor SMD 0603, reflow soldering, Vishay (see dcrcw.pdf)")
+    (tags "resistor 0603")
+    (attr smd)
+    (fp_text reference R26 (at 0 -1.45 45) (layer F.SilkS)
+      (effects (font (size 1 1) (thickness 0.15)))
+    )
+    (fp_text value 33 (at 0 1.5 45) (layer F.Fab)
+      (effects (font (size 1 1) (thickness 0.15)))
+    )
+    (fp_text user %R (at 0 -1.45 45) (layer F.Fab)
+      (effects (font (size 1 1) (thickness 0.15)))
+    )
+    (fp_line (start -0.8 0.4) (end -0.8 -0.4) (layer F.Fab) (width 0.1))
+    (fp_line (start 0.8 0.4) (end -0.8 0.4) (layer F.Fab) (width 0.1))
+    (fp_line (start 0.8 -0.4) (end 0.8 0.4) (layer F.Fab) (width 0.1))
+    (fp_line (start -0.8 -0.4) (end 0.8 -0.4) (layer F.Fab) (width 0.1))
+    (fp_line (start 0.5 0.68) (end -0.5 0.68) (layer F.SilkS) (width 0.12))
+    (fp_line (start -0.5 -0.68) (end 0.5 -0.68) (layer F.SilkS) (width 0.12))
+    (fp_line (start -1.25 -0.7) (end 1.25 -0.7) (layer F.CrtYd) (width 0.05))
+    (fp_line (start -1.25 -0.7) (end -1.25 0.7) (layer F.CrtYd) (width 0.05))
+    (fp_line (start 1.25 0.7) (end 1.25 -0.7) (layer F.CrtYd) (width 0.05))
+    (fp_line (start 1.25 0.7) (end -1.25 0.7) (layer F.CrtYd) (width 0.05))
+    (pad 1 smd rect (at -0.75 0 45) (size 0.5 0.9) (layers F.Cu F.Paste F.Mask)
+      (net 4 +3V3))
+    (pad 2 smd rect (at 0.75 0 45) (size 0.5 0.9) (layers F.Cu F.Paste F.Mask)
+      (net 1 VCC))
+    (model Resistors_SMD.3dshapes/R_0603.wrl
+      (at (xyz 0 0 0))
+      (scale (xyz 1 1 1))
+      (rotate (xyz 0 0 0))
+    )
+  )
   (gr_text "T R G" (at 138.684 115.824 340) (layer F.SilkS)
     (effects (font (size 1 1) (thickness 0.2)))
@@
   (gr_line (start 141.1732 89.8779) (end 141.1732 130.7719) (angle 90) (layer Dwgs.User) (width 0.2))
   (gr_line (start 163.9316 109.4994) (end 120.3706 109.4994) (angle 90) (layer Dwgs.User) (width 0.2))
+  (segment (start 155.974701 117.067228) (end 155.967532 117.067228) (width 0.6) (layer F.Cu) (net 1))
+  (segment (start 155.967532 117.067228) (end 155.01313 118.02163) (width 0.6) (layer F.Cu) (net 1))
   (segment (start 134.84 105.09) (end 134.57 105.09) (width 0.4) (layer F.Cu) (net 1))
   (segment (start 151.77 107.564) (end 151.384 107.95) (width 0.7) (layer B.Cu) (net 1))
@@
   (segment (start 155.597473 116.69) (end 155.974701 117.067228) (width 0.6) (layer F.Cu) (net 1))
   (segment (start 155.702 112.93) (end 156.31 112.93) (width 0.6) (layer F.Cu) (net 1))
-  (segment (start 155.974701 117.067228) (end 155.125998 117.804002) (width 0.6) (layer F.Cu) (net 1))
   (segment (start 156.517521 115.868135) (end 155.974701 117.067228) (width 0.6) (layer F.Cu) (net 1))
   (segment (start 156.91 114.69) (end 156.517521 115.868135) (width 0.6) (layer F.Cu) (net 1))
@@
   (segment (start 136.97 122.16) (end 137.59 122.16) (width 0.4) (layer F.Cu) (net 3))
   (segment (start 137.59 122.16) (end 137.81 121.94) (width 0.4) (layer F.Cu) (net 3))
+  (segment (start 152.835998 119.295998) (end 153.738762 119.295998) (width 0.6) (layer F.Cu) (net 4))
+  (segment (start 152.92 119.38) (end 152.2 118.66) (width 0.6) (layer B.Cu) (net 4))
+  (via (at 152.2 118.66) (size 0.8) (drill 0.5) (layers F.Cu B.Cu) (net 4))
+  (segment (start 152.2 118.66) (end 152.835998 119.295998) (width 0.6) (layer F.Cu) (net 4))
+  (segment (start 152.92 120.5) (end 152.92 119.38) (width 0.6) (layer B.Cu) (net 4))
+  (segment (start 153.738762 119.295998) (end 153.95247 119.08229) (width 0.6) (layer F.Cu) (net 4))
   (segment (start 133.03 106.4) (end 133.95 106.4) (width 0.6) (layer B.Cu) (net 4))
   (segment (start 133.03 106.4) (end 131.931363 106.4) (width 0.6) (layer B.Cu) (net 4))
@@
   (segment (start 137.62 101.4) (end 136.73 101.4) (width 0.6) (layer B.Cu) (net 4))
   (segment (start 136.73 101.4) (end 135.41 102.72) (width 0.6) (layer B.Cu) (net 4))
-  (segment (start 152.92 120.5) (end 152.92 119.38) (width 0.6) (layer B.Cu) (net 4))
-  (segment (start 152.835998 119.295998) (end 153.634002 119.295998) (width 0.6) (layer F.Cu) (net 4))
-  (segment (start 152.2 118.66) (end 152.835998 119.295998) (width 0.6) (layer F.Cu) (net 4))
-  (via (at 152.2 118.66) (size 0.8) (drill 0.5) (layers F.Cu B.Cu) (net 4))
-  (segment (start 152.92 119.38) (end 152.2 118.66) (width 0.6) (layer B.Cu) (net 4))
   (segment (start 136.86 101.01) (end 137.576 101.318) (width 0.6) (layer F.Cu) (net 4))
   (segment (start 137.62 101.4) (end 137.52 101.3) (width 0.6) (layer B.Cu) (net 4))
@@
   (segment (start 138.83 125.84) (end 143.08 125.87) (width 0.7) (layer B.Cu) (net 4))
   (segment (start 136.49 125.31) (end 138.83 125.84) (width 0.6) (layer B.Cu) (net 4))
-  (segment (start 153.634002 119.335998) (end 153.634002 119.295998) (width 0.6) (layer F.Cu) (net 4))
   (segment (start 135.94 120.09) (end 133.36 120.09) (width 0.6) (layer B.Cu) (net 4))
   (segment (start 135.89 120.14) (end 135.94 120.09) (width 0.4) (layer F.Cu) (net 4))
